File: 2110_LOW_THRESHOLD_SHORT_CHECKER.sch (KiCad schematic (older format))
At the start: 24 parts, among them CN2 2PIN, IC11 AD823AN, SW1 SS12D01G4

Commit message: 一部回路と、パターンの修正。
Parts:
- removed IC11: AD823AN, AD823AN:AD823AN, symbol 2110_LOW_THRESHOLD_SHORT_CHECKER-rescue:4558-IC
- added IC11: AD823AN, footprint:ic_DIP-8_W7.62mm, symbol IC:4558
- BT1, CN2: symbol 2110_LOW_THRESHOLD_SHORT_CHECKER-rescue:2PIN-connectors -> 2110_LOW_THRESHOLD_SHORT_CHECKER-rescue:2PIN-connectors-2110_LOW_THRESHOLD_SHORT_CHECKER-rescue
- BZ1: symbol 2110_LOW_THRESHOLD_SHORT_CHECKER-rescue:BUZZER-SPEAKER -> 2110_LOW_THRESHOLD_SHORT_CHECKER-rescue:BUZZER-SPEAKER-2110_LOW_THRESHOLD_SHORT_CHECKER-rescue
- C1, C2: symbol 2110_LOW_THRESHOLD_SHORT_CHECKER-rescue:C_Small-capacitor -> 2110_LOW_THRESHOLD_SHORT_CHECKER-rescue:C_Small-capacitor-2110_LOW_THRESHOLD_SHORT_CHECKER-rescue
- C3: symbol 2110_LOW_THRESHOLD_SHORT_CHECKER-rescue:CP1_Small-capacitor -> 2110_LOW_THRESHOLD_SHORT_CHECKER-rescue:CP1_Small-capacitor-2110_LOW_THRESHOLD_SHORT_CHECKER-rescue
- D1, D3, D4, D5, D6: symbol 2110_LOW_THRESHOLD_SHORT_CHECKER-rescue:DIODE-diode -> 2110_LOW_THRESHOLD_SHORT_CHECKER-rescue:DIODE-diode-2110_LOW_THRESHOLD_SHORT_CHECKER-rescue
- D2: symbol 2110_LOW_THRESHOLD_SHORT_CHECKER-rescue:LED-LED -> 2110_LOW_THRESHOLD_SHORT_CHECKER-rescue:LED-LED-2110_LOW_THRESHOLD_SHORT_CHECKER-rescue
- R1, R10, R2, R3, R4, R5, R6, R7, R8, R9: symbol 2110_LOW_THRESHOLD_SHORT_CHECKER-rescue:R-register -> 2110_LOW_THRESHOLD_SHORT_CHECKER-rescue:R-register-2110_LOW_THRESHOLD_SHORT_CHECKER-rescue
Connections:
- net +9V: now also SW1.2 (B), IC11.8 (V+), IC11.8 (V+); no longer SW1.1 (A)
- net GND: now also IC11.4 (V-), IC11.4 (V-)
- net at BT1.1: now also SW1.1 (A); no longer SW1.2 (B)
- net at R1.1, R2.2, R6.1: now also D5.1, D6.2, IC11.1
- net at R10.1, R8.2: now also IC11.5 (+)
- net at D3.2, D4.1, R7.2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: now also IC11.6 (-)
- net at D1.2: now also IC11.7
- net at C2.1, D1.1, R6.2: now also IC11.2 (-)
- net at R1.2, R3.2, R4.1: now also IC11.3 (+)
- no-connect marks 3 -> 1
Other:
- moved on the sheet: BZ1, D5, D6, R1, R2, R6, SW1
